File: i2s_tx.kicad_pcb (KiCad board)
At the start: 2 copper layers, 48.3 x 63.5 mm, 18 parts, among them IC1 AM26C31, IC2 AM26C31, IC3 AM26C31, J1 CONN_02x06, J2 CONN_01x07, J3 RJ45_Shielded, J4 RJ45_Shielded, J5 RJ45_Shielded, J6 CONN_01x02

Commit message: -- updated vias
Routing:
- net GND: track 55.4 -> 56.9 mm
Changed lines of the file:
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@@
     (thickness 1.6)
     (drawings 10)
-    (tracks 342)
+    (tracks 344)
     (zones 0)
     (modules 18)
@@
   )
   (setup
-    (last_trace_width 0.25)
+    (last_trace_width 0.5)
     (user_trace_width 0.25)
     (user_trace_width 0.5)
@@
   (segment (start 65.03 77.845) (end 63.645 79.23) (width 1) (layer F.Cu) (net 1))
   (segment (start 60.96 79.23) (end 58.42 79.23) (width 1) (layer F.Cu) (net 1))
-  (via (at 58.42 77.47) (size 1.5) (drill 1) (layers F.Cu B.Cu) (net 1))
-  (segment (start 58.42 79.23) (end 58.42 77.47) (width 1) (layer F.Cu) (net 1))
   (segment (start 49.53 63.01) (end 46.99 63.01) (width 1) (layer F.Cu) (net 1))
-  (via (at 46.99 65.405) (size 1.5) (drill 1) (layers F.Cu B.Cu) (net 1))
-  (segment (start 46.99 63.01) (end 46.99 65.405) (width 1) (layer F.Cu) (net 1))
-  (via (at 55.245 71.12) (size 1.5) (drill 1) (layers F.Cu B.Cu) (net 1))
+  (via (at 46.99 65.405) (size 0.8) (drill 0.4) (layers F.Cu B.Cu) (net 1))
+  (via (at 55.245 71.12) (size 0.8) (drill 0.4) (layers F.Cu B.Cu) (net 1))
   (segment (start 52.575 71.12) (end 55.245 71.12) (width 0.5) (layer F.Cu) (net 1))
-  (via (at 55.245 76.2) (size 1.5) (drill 1) (layers F.Cu B.Cu) (net 1))
+  (via (at 55.245 76.2) (size 0.8) (drill 0.4) (layers F.Cu B.Cu) (net 1))
   (segment (start 52.575 76.2) (end 55.245 76.2) (width 0.5) (layer F.Cu) (net 1))
-  (via (at 45.085 74.93) (size 1.5) (drill 1) (layers F.Cu B.Cu) (net 1))
+  (via (at 45.085 74.93) (size 0.8) (drill 0.4) (layers F.Cu B.Cu) (net 1))
   (segment (start 47.625 74.93) (end 45.085 74.93) (width 0.5) (layer F.Cu) (net 1))
   (segment (start 49.53 83.965) (end 46.99 83.965) (width 0.5) (layer F.Cu) (net 1))
-  (via (at 52.07 83.82) (size 1.5) (drill 1) (layers F.Cu B.Cu) (net 1))
+  (via (at 52.07 83.82) (size 0.8) (drill 0.4) (layers F.Cu B.Cu) (net 1))
   (segment (start 49.53 83.965) (end 51.925 83.965) (width 0.5) (layer F.Cu) (net 1))
   (segment (start 51.925 83.965) (end 52.07 83.82) (width 0.5) (layer F.Cu) (net 1))
-  (via (at 48.895 45.085) (size 1.5) (drill 1) (layers F.Cu B.Cu) (net 1))
+  (via (at 48.895 45.085) (size 0.8) (drill 0.4) (layers F.Cu B.Cu) (net 1))
   (segment (start 48.895 43.325) (end 48.895 45.085) (width 0.5) (layer F.Cu) (net 1))
-  (via (at 55.245 29.21) (size 1.5) (drill 1) (layers F.Cu B.Cu) (net 1))
+  (via (at 55.245 29.21) (size 0.8) (drill 0.4) (layers F.Cu B.Cu) (net 1))
   (segment (start 52.575 29.21) (end 55.245 29.21) (width 0.5) (layer F.Cu) (net 1))
-  (via (at 55.245 34.29) (size 1.5) (drill 1) (layers F.Cu B.Cu) (net 1))
+  (via (at 55.245 34.29) (size 0.8) (drill 0.4) (layers F.Cu B.Cu) (net 1))
   (segment (start 52.575 34.29) (end 55.245 34.29) (width 0.5) (layer F.Cu) (net 1))
-  (via (at 45.085 33.02) (size 1.5) (drill 1) (layers F.Cu B.Cu) (net 1))
+  (via (at 45.085 33.02) (size 0.8) (drill 0.4) (layers F.Cu B.Cu) (net 1))
   (segment (start 47.625 33.02) (end 45.085 33.02) (width 0.5) (layer F.Cu) (net 1))
-  (via (at 55.245 50.165) (size 1.5) (drill 1) (layers F.Cu B.Cu) (net 1))
+  (via (at 55.245 50.165) (size 0.8) (drill 0.4) (layers F.Cu B.Cu) (net 1))
   (segment (start 52.64 50.165) (end 55.245 50.165) (width 0.5) (layer F.Cu) (net 1))
-  (via (at 55.245 55.245) (size 1.5) (drill 1) (layers F.Cu B.Cu) (net 1))
+  (via (at 55.245 55.245) (size 0.8) (drill 0.4) (layers F.Cu B.Cu) (net 1))
   (segment (start 52.64 55.245) (end 55.245 55.245) (width 0.5) (layer F.Cu) (net 1))
   (segment (start 47.69 53.975) (end 45.085 53.975) (width 0.5) (layer F.Cu) (net 1))
-  (via (at 45.085 53.975) (size 1.5) (drill 1) (layers F.Cu B.Cu) (net 1))
+  (via (at 45.085 53.975) (size 0.8) (drill 0.4) (layers F.Cu B.Cu) (net 1))
   (segment (start 47.48 43.18) (end 46.355 42.055) (width 0.5) (layer F.Cu) (net 1))
   (segment (start 48.895 43.18) (end 47.48 43.18) (width 0.5) (layer F.Cu) (net 1))
+  (segment (start 46.99 63.01) (end 46.99 65.405) (width 0.5) (layer F.Cu) (net 1))
+  (segment (start 58.42 79.23) (end 58.42 77.47) (width 1) (layer F.Cu) (net 1))
+  (segment (start 59.182 76.708) (end 59.563 76.708) (width 1) (layer F.Cu) (net 1))
+  (segment (start 58.42 77.47) (end 59.182 76.708) (width 1) (layer F.Cu) (net 1))
+  (via (at 59.563 76.708) (size 2) (drill 1) (layers F.Cu B.Cu) (net 1))
   (segment (start 52.575 80.01) (end 53.34 80.01) (width 0.25) (layer F.Cu) (net 2))
   (segment (start 69.755 55.085) (end 69.85 54.99) (width 0.5) (layer F.Cu) (net 2))
@@
   (segment (start 67.31 52.545) (end 69.175001 54.410001) (width 0.25) (layer F.Cu) (net 2))
   (segment (start 69.175001 55.759999) (end 69.85 55.085) (width 0.25) (layer F.Cu) (net 2))
+  (segment (start 53.65 80.01) (end 59.055 74.605) (width 0.25) (layer F.Cu) (net 2))
   (segment (start 52.575 80.01) (end 53.65 80.01) (width 0.25) (layer F.Cu) (net 2))
   (segment (start 59.055 74.605) (end 59.055 60.22975) (width 0.25) (layer F.Cu) (net 2))
-  (segment (start 53.65 80.01) (end 59.055 74.605) (width 0.25) (layer F.Cu) (net 2))
   (segment (start 59.055 60.22975) (end 61.49975 57.785) (width 0.25) (layer F.Cu) (net 2))
   (segment (start 61.49975 57.785) (end 67.15 57.785) (width 0.25) (layer F.Cu) (net 2))
