File: i2s_tx.sch (KiCad schematic (older format))
At the start: 18 parts, among them IC1 AM26C31, IC2 AM26C31, IC3 AM26C31, J1 CONN_02x06, J2 CONN_02x06, J3 RJ45_Shielded, J4 RJ45_Shielded, J5 RJ45_Shielded, J6 CONN_01x02

Commit message: -- update
Parts:
- removed J2: CONN_02x06, Connector_PinHeader_2.00mm:PinHeader_2x06_P2.00mm_Vertical, symbol agg:CONN_02x06
- added J2: CONN_01x07, Connector_PinHeader_2.00mm:PinHeader_1x07_P2.00mm_Vertical, symbol agg:CONN_01x07
Connections:
- net GND: now also J2.7
- net I2S_IN_12: now also J2.1
- net I2S_IN_34: now also J2.2
- net I2S_IN_56: now also J2.3
- net I2S_IN_78: now also J2.4
- net I2S_SCLK: now also J2.5
- net I2S_WS: now also J2.6
Changed lines of the file:
@@
 Text GLabel 1500 5400 0    50   Input ~ 0
 I2S_OUT_78
-$Comp
-L agg:CONN_02x06 J2
-U 1 1 5CFBAA51
-P 1450 2250
-F 0 "J2" H 1400 2465 50  0000 C CNN
-F 1 "CONN_02x06" H 1400 2374 50  0000 C CNN
-F 2 "Connector_PinHeader_2.00mm:PinHeader_2x06_P2.00mm_Vertical" H 1450 2250 50  0001 C CNN
-F 3 "" H 1450 2250 50  0001 C CNN
-	1    1450 2250
-	1    0    0    -1
-$EndComp
 Wire Wire Line
 	1550 2250 1600 2250
@@
 L power:GND #PWR03
 U 1 1 5CFBAA6B
-P 1100 2800
-F 0 "#PWR03" H 1100 2550 50  0001 C CNN
-F 1 "GND" H 1105 2627 50  0000 C CNN
-F 2 "" H 1100 2800 50  0001 C CNN
-F 3 "" H 1100 2800 50  0001 C CNN
-	1    1100 2800
+P 1650 2900
+F 0 "#PWR03" H 1650 2650 50  0001 C CNN
+F 1 "GND" H 1655 2727 50  0000 C CNN
+F 2 "" H 1650 2900 50  0001 C CNN
+F 3 "" H 1650 2900 50  0001 C CNN
+	1    1650 2900
 	1    0    0    -1
 $EndComp
-Wire Wire Line
-	1100 2750 1100 2800
-Wire Wire Line
-	1100 2750 1250 2750
 Text GLabel 1600 2250 2    50   Input ~ 0
 I2S_IN_12
@@
 Text GLabel 3050 1200 1    50   Input ~ 0
 +5V
+$Comp
+L agg:CONN_01x07 J2
+U 1 1 5CF9C40C
+P 1450 2250
+F 0 "J2" H 1483 2465 50  0000 C CNN
+F 1 "CONN_01x07" H 1483 2374 50  0000 C CNN
+F 2 "Connector_PinHeader_2.00mm:PinHeader_1x07_P2.00mm_Vertical" H 1450 2250 50  0001 C CNN
+F 3 "" H 1450 2250 50  0001 C CNN
+	1    1450 2250
+	1    0    0    -1
+$EndComp
+Wire Wire Line
+	1650 2900 1650 2850
+Wire Wire Line
+	1650 2850 1550 2850
 $EndSCHEMATC

Commit message: -- update
Parts:
- C7: value CP_Small -> 10µF
Changed lines of the file:
@@
 P 2700 1300
 F 0 "C7" H 2788 1346 50  0000 L CNN
-F 1 "CP_Small" H 2788 1255 50  0000 L CNN
+F 1 "10µF" H 2788 1255 50  0000 L CNN
 F 2 "Capacitor_SMD:CP_Elec_6.3x5.4" H 2700 1300 50  0001 C CNN
 F 3 "~" H 2700 1300 50  0001 C CNN
